Commit message: trajectory plugin

File: src/rrbot_description/urdf/rrbot.description.xacro (robot description, xacro)
@@ -43,5 +43,5 @@
     <origin xyz="0 ${width} ${height1 - axel_offset}" rpy="0 0 0"/>
     <axis xyz="0 1 0"/>
-    <dynamics damping="0.7"/>
+    <dynamics damping="10.0"  friction="10.0"/>
   </joint>
   <!-- Middle Link -->
@@ -74,5 +74,5 @@
     <origin xyz="0 ${width} ${height2 - axel_offset*2}" rpy="0 0 0"/>
     <axis xyz="0 1 0"/>
-    <dynamics damping="0.7"/>
+    <dynamics damping="10.0"  friction="10.0"/>
   </joint>
   <!-- Top Link -->

File: src/rrbot_description/urdf/rrbot.gazebo.xacro (robot description, xacro)
@@ -4,5 +4,5 @@
 https://github.com/ros-simulation/gazebo_ros_demos/blob/kinetic-devel/rrbot_description/urdf/materials.xacro
 -->
-<robot params="prefix">
+<robot >
     <gazebo>
         <plugin name="gazebo_ros_joint_state_publisher"
@@ -13,9 +13,18 @@
         </plugin>
     </gazebo>
-    <gazebo reference="${prefix}base_link">
+    <gazebo>
+        <plugin name="gazebo_ros_joint_pose_trajectory"
+            filename="libgazebo_ros_joint_pose_trajectory.so">
+            <update_rate>2</update_rate>
+        </plugin>
+    </gazebo>
+    <gazebo reference="base_link">
         <material>Gazebo/Black</material>
       </gazebo>
-      <gazebo reference="${prefix}link1">
+      <gazebo reference="link1">
         <material>Gazebo/Orange</material>
       </gazebo>
 </robot>
+<!--
+ros2 topic pub -1 /set_joint_trajectory trajectory_msgs/msg/JointTrajectory  '{header: {frame_id: world}, joint_names: [joint1, joint2], points: [  {positions: {1,1}} ]}'
+ -->

Commit message: bk

File: src/rrbot_description/urdf/rrbot.description.xacro (robot description, xacro)
@@ -108,4 +108,12 @@
   <link name="${prefix}tool_link">
   </link>
+  <!-- imu link -->
+  <link name="${prefix}imu_link">
+  </link>
+  <joint name="${prefix}imu_link" type="fixed">
+    <origin xyz="0 0.1 1" rpy="0 0 0" />
+    <parent link="${prefix}link2"/>
+    <child link="${prefix}imu_link" />
+  </joint>
   </xacro:macro>
 </robot>

File: src/rrbot_description/urdf/rrbot.gazebo.xacro (robot description, xacro)
@@ -25,4 +25,10 @@
         <material>Gazebo/Orange</material>
       </gazebo>
+      <gazebo reference="imu_link">
+        <sensor name="imu_sensor" type="imu">
+          <always_on>true</always_on>
+          <update_rate>30</update_rate>
+        </sensor>
+      </gazebo>
 </robot>
 <!--

File: src/rrbot_description/urdf/rrbot.ros_control.xacro (robot description, xacro)
@@ -12,8 +12,20 @@
             <state_interface name="position" />
         </joint>
+        <sensor name="imu_sensor">
+            <state_interface name="orientation.x"/>
+            <state_interface name="orientation.y"/>
+            <state_interface name="orientation.z"/>
+            <state_interface name="orientation.w"/>
+            <state_interface name="angular_velocity.x"/>
+            <state_interface name="angular_velocity.y"/>
+            <state_interface name="angular_velocity.z"/>
+            <state_interface name="linear_acceleration.x"/>
+            <state_interface name="linear_acceleration.y"/>
+            <state_interface name="linear_acceleration.z"/>
+        </sensor>
     </ros2_control>
     <gazebo>
         <plugin filename="libgazebo_ros2_control.so" name="gazebo_ros2_control">
-            <parameters>$(find rrbot_bringup)/config/position_and_effort.yaml</parameters>
+            <parameters>$(find rrbot_bringup)/config/position_and_effort_imu.yaml</parameters>
         </plugin>
     </gazebo>
